File: Eurorack Power.kicad_sch (KiCad schematic)
At the start: 3 parts, among them J1 IDC_2x05

Commit message: Added pcb for v0.1
Parts:
- J1: Manufacturers Name XKB Connectivity -> XKB Connectivity
Changed lines of the file:
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@@
       (effects (font (size 1.27 1.27)) hide)
     )
-    (property "Manufacturers Name" "XKB Connectivity " (id 6) (at 27.94 38.1 0)
+    (property "Manufacturers Name" "XKB Connectivity" (id 6) (at 27.94 38.1 0)
       (effects (font (size 1.27 1.27)) hide)
     )
