File: MiniAttenuMix.kicad_sch (KiCad schematic)
At the start: 32 parts, among them U1 TL074, U2 TL074

Commit message: Added pcb for v0.1
Parts:
- removed U1, U2: TL074, symbol Amplifier_Operational:TL074
- added IN5: PJ-3001F, benjiaomodular:AudioJack_3.5mm, symbol Connector:AudioJack2_SwitchT
- added R10, R5: 20k, Resistor_SMD:R_0603_1608Metric_Pad0.98x0.95mm_HandSolder, symbol Device:R
- added R14: 100k, Resistor_SMD:R_0603_1608Metric_Pad0.98x0.95mm_HandSolder, symbol Device:R
- added U1, U2: TL072, Package_SO:SOIC-8_3.9x4.9mm_P1.27mm, symbol Amplifier_Operational:TL072
- added U3: TL074, Package_SO:SOIC-14_3.9x8.7mm_P1.27mm, symbol Amplifier_Operational:TL074
- D1: footprint (none) -> LED_THT:LED_D3.0mm; Manufacturers Name (none) -> KENTO; Manufacturers Part Number (none) -> 3ARG4HWC
- IN1, IN2, IN3, IN4, OUT1, OUT_INV1: footprint (none) -> benjiaomodular:AudioJack_3.5mm; Manufacturers Name (none) -> Tayda Electronics; Manufacturers Part Number (none) -> PJ-3001F
- R1, R2, R3, R4: footprint (none) -> Resistor_SMD:R_0603_1608Metric_Pad0.98x0.95mm_HandSolder; Manufacturers Name (none) -> YAGEO; Manufacturers Part Number (none) -> RC0603FR-0720KL
- R11: renamed from R9; footprint (none) -> Resistor_SMD:R_0603_1608Metric_Pad0.98x0.95mm_HandSolder; Manufacturers Name (none) -> YAGEO; Manufacturers Part Number (none) -> RC0603FR-07100KL
- R12: renamed from R10; footprint (none) -> Resistor_SMD:R_0603_1608Metric_Pad0.98x0.95mm_HandSolder; Manufacturers Name (none) -> YAGEO; Manufacturers Part Number (none) -> RC0603FR-07100KL
- R13: renamed from R11; footprint (none) -> Resistor_SMD:R_0603_1608Metric_Pad0.98x0.95mm_HandSolder; Manufacturers Name (none) -> YAGEO; Manufacturers Part Number (none) -> RC0603FR-07100KL
- R15: renamed from R12; footprint (none) -> Resistor_SMD:R_0603_1608Metric_Pad0.98x0.95mm_HandSolder; Manufacturers Name (none) -> YAGEO; Manufacturers Part Number (none) -> RC0603FR-07100KL
- R16: renamed from R13; footprint (none) -> Resistor_SMD:R_0603_1608Metric_Pad0.98x0.95mm_HandSolder; Manufacturers Name (none) -> YAGEO; Manufacturers Part Number (none) -> RC0603FR-07100KL
- R17: renamed from R14; footprint (none) -> Resistor_SMD:R_0603_1608Metric_Pad0.98x0.95mm_HandSolder; Manufacturers Name (none) -> YAGEO; Manufacturers Part Number (none) -> RC0603FR-07100KL
- R18: renamed from R15; footprint (none) -> Resistor_SMD:R_0603_1608Metric_Pad0.98x0.95mm_HandSolder; Manufacturers Name (none) -> YAGEO; Manufacturers Part Number (none) -> RC0603FR-07100KL
- R19: renamed from R16; footprint (none) -> Resistor_SMD:R_0603_1608Metric_Pad0.98x0.95mm_HandSolder; Manufacturers Name (none) -> YAGEO; Manufacturers Part Number (none) -> RC0603FR-074K7L
- R20: renamed from R17; footprint (none) -> Resistor_SMD:R_0603_1608Metric_Pad0.98x0.95mm_HandSolder; Manufacturers Name (none) -> YAGEO; Manufacturers Part Number (none) -> RC0603FR-071KL
- R21: renamed from R18; footprint (none) -> Resistor_SMD:R_0603_1608Metric_Pad0.98x0.95mm_HandSolder; Manufacturers Name (none) -> YAGEO; Manufacturers Part Number (none) -> RC0603FR-071KL
- R6: renamed from R5; footprint (none) -> Resistor_SMD:R_0603_1608Metric_Pad0.98x0.95mm_HandSolder; Manufacturers Name (none) -> YAGEO; Manufacturers Part Number (none) -> RC0603FR-0720KL
- R7: renamed from R6; footprint (none) -> Resistor_SMD:R_0603_1608Metric_Pad0.98x0.95mm_HandSolder; Manufacturers Name (none) -> YAGEO; Manufacturers Part Number (none) -> RC0603FR-0720KL
- R8: renamed from R7; footprint (none) -> Resistor_SMD:R_0603_1608Metric_Pad0.98x0.95mm_HandSolder; Manufacturers Name (none) -> YAGEO; Manufacturers Part Number (none) -> RC0603FR-0720KL
- R9: renamed from R8; footprint (none) -> Resistor_SMD:R_0603_1608Metric_Pad0.98x0.95mm_HandSolder; Manufacturers Name (none) -> YAGEO; Manufacturers Part Number (none) -> RC0603FR-0720KL
- RV1, RV2, RV3, RV4, RV5: footprint (none) -> benjiaomodular:Potentiometer_RV09; Manufacturers Name (none) -> Alpha (Taiwan); Manufacturers Part Number (none) -> RD901F-40-15R1-B100K
Connections:
- net GND: now also IN2.S, IN3.S, RV3.3, RV4.3, RV5.3, IN5.S, IN5.TN, U3.12 (+), U3.3 (+); no longer RV3.1, RV4.1, RV5.1
- net NEG_12V: now also U1.4 (V-), U2.4 (V-), U3.11 (V-)
- net POS_12V: now also U1.8 (V+), U2.8 (V+), U3.4 (V+)
- net at R11.1, R7.2: now also U1.7
- net at R11.2, R12.2, R13.2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: now also R14.2, U3.2 (-)
- net at R17.2, R18.1: now also U3.10 (+), U3.13 (-)
- net at R18.2, R21.1: now also U3.14
- net at R19.2: now also U3.8, U3.9 (-)
- net at R17.1: now also R16.2, R20.1, U3.1; no longer RV5.2
- net at RV2.2: now also U1.5 (+)
- net at R15.1, R6.2: now also U1.1
- net at RV3.2: now also U2.3 (+)
- net at IN3.T, R3.1: now also RV3.1; no longer RV3.3
- net at IN4.T, R4.1: now also RV4.1; no longer RV4.3
- net at R2.2, R7.1: now also U1.6 (-)
- net at R3.2, R8.1: now also U2.2 (-)
- net at R12.1, R8.2: now also U2.1
- net at RV4.2: now also U2.5 (+)
- net at R4.2, R9.1: now also U2.6 (-)
- net at R13.1, R9.2: now also U2.7
- net at R1.2, R6.1: now also U1.2 (-)
- net at RV1.2: now also U1.3 (+)
- new net: IN5.T, R5.1, RV5.1
- new net: R10.1, R5.2, U3.6 (-)
- new net: R10.2, R14.1, U3.7
- new net: RV5.2, U3.5 (+)
Other:
- moved on the sheet: OUT_INV1, R20
