File: MiniAttenuMix/MiniAttenuMix v0.2/Eurorack Power.kicad_sch (KiCad schematic)
At the start: 3 parts, among them J1 IDC_2x05

Commit message: Added v0.2 gerbers
Parts:
- removed C1, C2: 22uF, Capacitor_SMD:C_0805_2012Metric_Pad1.18x1.45mm_HandSolder, symbol MiniDelay-rescue:CP1-Device
- added C1, C2: 22uF, Capacitor_SMD:C_0805_2012Metric_Pad1.18x1.45mm_HandSolder, symbol Device:C_Polarized_US
Connections:
- net +12V: now also C1.1
- net -12V: now also C2.2
- net GND: now also C1.2, C2.1
Changed lines of the file:
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@@
   (junction (at 33.02 35.56) (diameter 0) (color 0 0 0 0)
   )
+  (junction (at 45.72 26.67) (diameter 0) (color 0 0 0 0)
+  )
   (junction (at 35.56 36.576) (diameter 0) (color 0 0 0 0)
   )
@@
   (junction (at 33.02 46.99) (diameter 0) (color 0 0 0 0)
   )
+  (junction (at 45.974 46.99) (diameter 0) (color 0 0 0 0)
+  )
   (junction (at 33.02 36.576) (diameter 0) (color 0 0 0 0)
   )
@@
     (stroke (width 0) (type default) (color 0 0 0 0))
   )
-  (wire (pts (xy 41.656 26.67) (xy 48.514 26.67))
+  (wire (pts (xy 41.656 26.67) (xy 45.72 26.67))
     (stroke (width 0) (type default) (color 0 0 0 0))
   )
@@
     (stroke (width 0) (type default) (color 0 0 0 0))
   )
+  (wire (pts (xy 45.974 46.99) (xy 48.514 46.99))
+    (stroke (width 0) (type default) (color 0 0 0 0))
+  )
   (wire (pts (xy 35.56 36.576) (xy 41.656 36.576))
     (stroke (width 0) (type default) (color 0 0 0 0))
   )
-  (wire (pts (xy 41.656 46.99) (xy 48.514 46.99))
+  (wire (pts (xy 41.656 46.99) (xy 45.974 46.99))
     (stroke (width 0) (type default) (color 0 0 0 0))
   )
   (wire (pts (xy 41.656 26.67) (xy 41.656 27.686))
+    (stroke (width 0) (type default) (color 0 0 0 0))
+  )
+  (wire (pts (xy 45.72 26.67) (xy 48.514 26.67))
     (stroke (width 0) (type default) (color 0 0 0 0))
   )
@@
     (pin "1")
   )
-  (symbol (lib_id "MiniDelay-rescue:CP1-Device") (at 41.656 41.656 0) (unit 1)
-    (in_bom yes) (on_board yes)
-    (property "Reference" "C2" (id 0) (at 44.577 40.4876 0)
-      (effects (font (size 1.27 1.27)) (justify left))
-    )
-    (property "Value" "22uF" (id 1) (at 44.577 42.799 0)
-      (effects (font (size 1.27 1.27)) (justify left))
-    )
-    (property "Footprint" "Capacitor_SMD:C_0805_2012Metric_Pad1.18x1.45mm_HandSolder" (id 2) (at 41.656 41.656 0)
-      (effects (font (size 1.27 1.27)) hide)
-    )
-    (property "Datasheet" "~" (id 3) (at 41.656 41.656 0)
-      (effects (font (size 1.27 1.27)) hide)
-    )
-    (property "LCSC Part #" "C49678" (id 4) (at 41.656 41.656 0)
-      (effects (font (size 1.27 1.27)) hide)
-    )
-    (property "Mfg #" "CC0805KRX7R9BB104" (id 5) (at 41.656 41.656 0)
-      (effects (font (size 1.27 1.27)) hide)
-    )
-    (property "Manufacturers Part Number" "CC0805KRX7R9BB104" (id 6) (at 41.656 41.656 0)
-      (effects (font (size 1.27 1.27)) hide)
-    )
-    (property "Manufacturers Name" "YAGEO" (id 7) (at 41.656 41.656 0)
-      (effects (font (size 1.27 1.27)) hide)
-    )
-    (property "Type" "Surface mount" (id 8) (at 41.656 41.656 0)
-      (effects (font (size 1.27 1.27)) hide)
-    )
-    (property "Package" "0805" (id 9) (at 41.656 41.656 0)
-      (effects (font (size 1.27 1.27)) hide)
-    )
-    (property "Part Description" "Multilayer Ceramic Capacitors MLCC - SMD/SMT 50 V 0.1uF X7R 0805 10% " (id 10) (at 41.656 41.656 0)
+  (symbol (lib_id "power:PWR_FLAG") (at 45.72 26.67 0) (unit 1)
+    (in_bom yes) (on_board yes) (fields_autoplaced)
+    (property "Reference" "#FLG0101" (id 0) (at 45.72 24.765 0)
+      (effects (font (size 1.27 1.27)) hide)
+    )
+    (property "Value" "PWR_FLAG" (id 1) (at 45.72 21.59 0))
+    (property "Footprint" "" (id 2) (at 45.72 26.67 0)
+      (effects (font (size 1.27 1.27)) hide)
+    )
+    (property "Datasheet" "~" (id 3) (at 45.72 26.67 0)
+      (effects (font (size 1.27 1.27)) hide)
+    )
+    (pin "1")
+  )
+  (symbol (lib_id "Device:C_Polarized_US") (at 41.656 31.496 0) (unit 1)
+    (in_bom yes) (on_board yes) (fields_autoplaced)
+    (property "Reference" "C1" (id 0) (at 45.72 29.5909 0)
+      (effects (font (size 1.27 1.27)) (justify left))
+    )
+    (property "Value" "22uF" (id 1) (at 45.72 32.1309 0)
+      (effects (font (size 1.27 1.27)) (justify left))
+    )
+    (property "Footprint" "Capacitor_SMD:C_0805_2012Metric_Pad1.18x1.45mm_HandSolder" (id 2) (at 41.656 31.496 0)
+      (effects (font (size 1.27 1.27)) hide)
+    )
+    (property "Datasheet" "~" (id 3) (at 41.656 31.496 0)
+      (effects (font (size 1.27 1.27)) hide)
+    )
+    (property "Manufacturers Name" "Murata Electronics " (id 4) (at 41.656 31.496 0)
+      (effects (font (size 1.27 1.27)) hide)
+    )
+    (property "Manufacturers Part Number" "GRM21BR61E226ME44L " (id 5) (at 41.656 31.496 0)
       (effects (font (size 1.27 1.27)) hide)
     )
@@
     (pin "1")
   )
-  (symbol (lib_id "power:PWR_FLAG") (at 41.656 36.576 270) (unit 1)
-    (in_bom yes) (on_board yes) (fields_autoplaced)
-    (property "Reference" "#FLG01" (id 0) (at 43.561 36.576 0)
-      (effects (font (size 1.27 1.27)) hide)
-    )
-    (property "Value" "PWR_FLAG" (id 1) (at 45.593 36.5759 90)
-      (effects (font (size 1.27 1.27)) (justify left) hide)
-    )
-    (property "Footprint" "" (id 2) (at 41.656 36.576 0)
-      (effects (font (size 1.27 1.27)) hide)
-    )
-    (property "Datasheet" "~" (id 3) (at 41.656 36.576 0)
+  (symbol (lib_id "power:PWR_FLAG") (at 45.974 46.99 180) (unit 1)
+    (in_bom yes) (on_board yes) (fields_autoplaced)
+    (property "Reference" "#FLG0102" (id 0) (at 45.974 48.895 0)
+      (effects (font (size 1.27 1.27)) hide)
+    )
+    (property "Value" "PWR_FLAG" (id 1) (at 47.752 48.2599 0)
+      (effects (font (size 1.27 1.27)) (justify right))
+    )
+    (property "Footprint" "" (id 2) (at 45.974 46.99 0)
+      (effects (font (size 1.27 1.27)) hide)
+    )
+    (property "Datasheet" "~" (id 3) (at 45.974 46.99 0)
       (effects (font (size 1.27 1.27)) hide)
     )
@@
     (pin "1")
   )
-  (symbol (lib_id "MiniDelay-rescue:CP1-Device") (at 41.656 31.496 0) (unit 1)
-    (in_bom yes) (on_board yes)
-    (property "Reference" "C1" (id 0) (at 44.577 30.3276 0)
-      (effects (font (size 1.27 1.27)) (justify left))
-    )
-    (property "Value" "22uF" (id 1) (at 44.577 32.639 0)
-      (effects (font (size 1.27 1.27)) (justify left))
-    )
-    (property "Footprint" "Capacitor_SMD:C_0805_2012Metric_Pad1.18x1.45mm_HandSolder" (id 2) (at 41.656 31.496 0)
-      (effects (font (size 1.27 1.27)) hide)
-    )
-    (property "Datasheet" "~" (id 3) (at 41.656 31.496 0)
-      (effects (font (size 1.27 1.27)) hide)
-    )
-    (property "LCSC Part #" "C49678" (id 4) (at 41.656 31.496 0)
-      (effects (font (size 1.27 1.27)) hide)
-    )
-    (property "Mfg #" "CC0805KRX7R9BB104" (id 5) (at 41.656 31.496 0)
-      (effects (font (size 1.27 1.27)) hide)
-    )
-    (property "Manufacturers Part Number" "CC0805KRX7R9BB104" (id 6) (at 41.656 31.496 0)
-      (effects (font (size 1.27 1.27)) hide)
-    )
-    (property "Manufacturers Name" "YAGEO" (id 7) (at 41.656 31.496 0)
-      (effects (font (size 1.27 1.27)) hide)
-    )
-    (property "Type" "Surface mount" (id 8) (at 41.656 31.496 0)
-      (effects (font (size 1.27 1.27)) hide)
-    )
-    (property "Package" "0805" (id 9) (at 41.656 31.496 0)
-      (effects (font (size 1.27 1.27)) hide)
-    )
-    (property "Part Description" "Multilayer Ceramic Capacitors MLCC - SMD/SMT 50 V 0.1uF X7R 0805 10% " (id 10) (at 41.656 31.496 0)
-      (effects (font (size 1.27 1.27)) hide)
-    )
+  (symbol (lib_id "power:PWR_FLAG") (at 41.656 36.576 270) (unit 1)
+    (in_bom yes) (on_board yes) (fields_autoplaced)
+    (property "Reference" "#FLG0103" (id 0) (at 43.561 36.576 0)
+      (effects (font (size 1.27 1.27)) hide)
+    )
+    (property "Value" "PWR_FLAG" (id 1) (at 45.7802 36.5759 90)
+      (effects (font (size 1.27 1.27)) (justify left))
+    )
+    (property "Footprint" "" (id 2) (at 41.656 36.576 0)
+      (effects (font (size 1.27 1.27)) hide)
+    )
+    (property "Datasheet" "~" (id 3) (at 41.656 36.576 0)
+      (effects (font (size 1.27 1.27)) hide)
+    )
+    (pin "1")
+  )
+  (symbol (lib_id "Device:C_Polarized_US") (at 41.656 41.656 0) (unit 1)
+    (in_bom yes) (on_board yes) (fields_autoplaced)
+    (property "Reference" "C2" (id 0) (at 45.72 39.7509 0)
+      (effects (font (size 1.27 1.27)) (justify left))
+    )
+    (property "Value" "22uF" (id 1) (at 45.72 42.2909 0)
+      (effects (font (size 1.27 1.27)) (justify left))
+    )
+    (property "Footprint" "Capacitor_SMD:C_0805_2012Metric_Pad1.18x1.45mm_HandSolder" (id 2) (at 41.656 41.656 0)
+      (effects (font (size 1.27 1.27)) hide)
+    )
+    (property "Datasheet" "~" (id 3) (at 41.656 41.656 0)
+      (effects (font (size 1.27 1.27)) hide)
+    )
+    (property "Manufacturers Name" "Murata Electronics " (id 4) (at 41.656 41.656 0)
+      (effects (font (size 1.27 1.27)) hide)
+    )
+    (property "Manufacturers Part Number" "GRM21BR61E226ME44L " (id 5) (at 41.656 41.656 0)
+      (effects (font (size 1.27 1.27)) hide)
+    )
