File: MiniAttenuMix/MiniAttenuMix v0.3/MiniAttenuMix.kicad_pcb (KiCad board)
At the start: 2 copper layers, 50 x 128.5 mm, 55 parts, among them J1 IDC_2x05, U1 TL072, U2 TL072, U3 TL074

Commit message: Added v0.3
Parts:
- R19: value 1k -> 330
- moved R19 6.66 mm to (147.8, 112.0), turned to 90 degrees
- moved R22 0.51 mm to (158.0, 133.6), turned to 0 degrees
Connections:
- R19 pad 1: Net-(D1-Pad2) -> Net-(R19-Pad1)
- R19 pad 2: Net-(R19-Pad2) -> Net-(D1-Pad1)
- R22 pad 1: Net-(D1-Pad1) -> Net-(D1-Pad2)
- U3 pad 8: Net-(D1-Pad1) -> Net-(R19-Pad1)
- U3 pad 9: Net-(R19-Pad2) -> Net-(D1-Pad2)
Routing:
- net Net-(R19-Pad2): track 26.8 -> 0.00 mm, vias 2 -> 0
- net Net-(D1-Pad2): track 2.08 -> 26.8 mm, vias 0 -> 1
- net Net-(D1-Pad1): track 26.2 -> 2.67 mm, vias 1 -> 0
- net Net-(R19-Pad1): track 0.00 -> 23.0 mm, vias 0 -> 2
- net Net-(U3-Pad10): track 34.7 -> 26.0 mm, vias 2 -> 0
- net POS_12V: track 189.4 -> 188.8 mm
Other:
- board text added: "MiniAttenuMix v0.3"
- board text removed: "MiniAttenuMix v0.2"
