File: MiniAttenuMix/MiniAttenuMix v0.3/MiniAttenuMix.kicad_sch (KiCad schematic)
At the start: 38 parts, among them U1 TL072, U2 TL072, U3 TL074

Commit message: Added v0.3
Parts:
- R19: value 1k -> 330; Manufacturers Name YAGEO -> TE Connectivity / Holsworthy; Manufacturers Part Number RC0603FR-071KL -> CRG0603F330R
- R22: Manufacturers Name YAGEO -> TE Connectivity / Holsworthy; Manufacturers Part Number RC0603FR-074K7L -> CRG0603F330R
Connections:
- net at R19.1: now also U3.8; no longer D1.2 (AK)
- net at R19.2: now also D1.1 (KA); no longer U3.9 (-)
- new net: D1.2 (AK), R22.1, U3.9 (-)
Other:
- moved on the sheet: D1, R19, R22
